File: PCB/schemat.sch (EAGLE design)
At the start: 54 parts, among them IC1 TEXAS_INSTRUMENTS_TLV3502AIDT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, IC2 74AC244DW, IC3 74AHC1G86DBV, IC4 7805DT

Commit message: Praca nad rozdziałem 3
Parts:
- D1: value (none) -> S1A
- FUSE: value (none) -> 750 mA
- R6: value 10k -> 5k1
Other:
- moved on the sheet: R7, R8, R9
Changed lines of the file:
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@@
 <?xml version="1.0" encoding="utf-8"?>
 <!DOCTYPE eagle SYSTEM "eagle.dtd">
-<eagle version="9.1.2">
+<eagle version="8.0.1">
 <drawing>
 <settings>
 <setting alwaysvectorfont="no"/>
-<setting keepoldvectorfont="yes"/>
 <setting verticaltext="up"/>
 </settings>
@@
 <part name="GND16" library="supply1" deviceset="GND" device=""/>
 <part name="P+5" library="supply1" deviceset="+5V" device=""/>
-<part name="D1" library="adafruit" deviceset="DIODE" device="SMA"/>
+<part name="D1" library="adafruit" deviceset="DIODE" device="SMA" value="S1A"/>
 <part name="PWR_SW" library="switch-misc" deviceset="9077-2" device="" value=""/>
 <part name="DC-IN" library="con-jack" deviceset="JACK-PLUG" device="1"/>
@@
 <part name="R8" library="resistor" deviceset="R-EU_" device="R1206" value="10k"/>
 <part name="P+8" library="supply1" deviceset="+5V" device=""/>
-<part name="FUSE" library="adafruit" deviceset="PTCFUSE" device="-1812"/>
+<part name="FUSE" library="adafruit" deviceset="PTCFUSE" device="-1812" value="750 mA"/>
 <part name="R1_A" library="pinhead" deviceset="PINHD-1X2" device=""/>
 <part name="R3_A" library="pinhead" deviceset="PINHD-1X2" device=""/>
@@
 <part name="GND20" library="supply1" deviceset="GND" device=""/>
 <part name="C3" library="resistor" deviceset="C-EU" device="C1206K" value="100nF"/>
-<part name="FINGERPAD" library="dom-key" deviceset="FINGERPAD-2B" device=""/>
+<part name="FINGERPAD" library="dom-key" deviceset="FINGERPAD-2B" device="" value=""/>
 <part name="LCD" library="pinhead" deviceset="PINHD-1X4" device=""/>
 <part name="P+6" library="supply1" deviceset="+5V" device=""/>
 <part name="GND11" library="supply1" deviceset="GND" device=""/>
-<part name="R6" library="resistor" deviceset="R-EU_" device="R1206" value="10k"/>
+<part name="R6" library="resistor" deviceset="R-EU_" device="R1206" value="5k1"/>
 <part name="GND10" library="supply1" deviceset="GND" device=""/>
 <part name="P+10" library="supply1" deviceset="+5V" device=""/>
@@
 <instance part="P+7" gate="1" x="234.95" y="172.72"/>
 <instance part="GND19" gate="1" x="234.95" y="139.7"/>
-<instance part="R7" gate="G$1" x="184.15" y="157.48" rot="R90"/>
-<instance part="R9" gate="G$1" x="194.31" y="157.48" rot="R90"/>
-<instance part="R8" gate="G$1" x="204.47" y="157.48" rot="R90"/>
-<instance part="P+8" gate="1" x="194.31" y="172.72"/>
+<instance part="R7" gate="G$1" x="207.01" y="157.48" rot="R90"/>
+<instance part="R9" gate="G$1" x="186.69" y="157.48" rot="R90"/>
+<instance part="R8" gate="G$1" x="196.85" y="157.48" rot="R90"/>
+<instance part="P+8" gate="1" x="196.85" y="172.72"/>
 <instance part="FUSE" gate="G$1" x="43.18" y="93.98"/>
 <instance part="LCD" gate="A" x="81.28" y="153.67"/>
@@
 <segment>
 <pinref part="R7" gate="G$1" pin="1"/>
-<wire x1="184.15" y1="152.4" x2="184.15" y2="149.86" width="0.1524" layer="91"/>
-<label x="184.15" y="149.86" size="2.54" layer="95" rot="R270" xref="yes"/>
+<wire x1="207.01" y1="152.4" x2="207.01" y2="149.86" width="0.1524" layer="91"/>
+<label x="207.01" y="149.86" size="2.54" layer="95" rot="R270" xref="yes"/>
 </segment>
 <segment>
@@
 </segment>
 <segment>
-<pinref part="P+8" gate="1" pin="+5V"/>
-<pinref part="R9" gate="G$1" pin="2"/>
-<wire x1="194.31" y1="170.18" x2="194.31" y2="165.1" width="0.1524" layer="91"/>
-<wire x1="194.31" y1="165.1" x2="194.31" y2="162.56" width="0.1524" layer="91"/>
-<wire x1="194.31" y1="165.1" x2="204.47" y2="165.1" width="0.1524" layer="91"/>
-<junction x="194.31" y="165.1"/>
-<pinref part="R8" gate="G$1" pin="2"/>
-<wire x1="204.47" y1="165.1" x2="204.47" y2="162.56" width="0.1524" layer="91"/>
-<wire x1="194.31" y1="165.1" x2="184.15" y2="165.1" width="0.1524" layer="91"/>
-<pinref part="R7" gate="G$1" pin="2"/>
-<wire x1="184.15" y1="165.1" x2="184.15" y2="162.56" width="0.1524" layer="91"/>
-</segment>
-<segment>
 <pinref part="LCD" gate="A" pin="1"/>
 <pinref part="P+6" gate="1" pin="+5V"/>
@@
 <pinref part="R5" gate="G$1" pin="2"/>
 <wire x1="11.43" y1="168.91" x2="11.43" y2="167.64" width="0.1524" layer="91"/>
+</segment>
+<segment>
+<pinref part="R9" gate="G$1" pin="2"/>
+<wire x1="186.69" y1="165.1" x2="186.69" y2="162.56" width="0.1524" layer="91"/>
+<wire x1="186.69" y1="165.1" x2="196.85" y2="165.1" width="0.1524" layer="91"/>
+<pinref part="R8" gate="G$1" pin="2"/>
+<wire x1="196.85" y1="165.1" x2="196.85" y2="162.56" width="0.1524" layer="91"/>
+<pinref part="R7" gate="G$1" pin="2"/>
+<wire x1="207.01" y1="162.56" x2="207.01" y2="165.1" width="0.1524" layer="91"/>
+<wire x1="207.01" y1="165.1" x2="196.85" y2="165.1" width="0.1524" layer="91"/>
+<pinref part="P+8" gate="1" pin="+5V"/>
+<wire x1="196.85" y1="170.18" x2="196.85" y2="165.1" width="0.1524" layer="91"/>
+<junction x="196.85" y="165.1"/>
 </segment>
 </net>
@@
 <segment>
 <pinref part="R8" gate="G$1" pin="1"/>
-<wire x1="204.47" y1="152.4" x2="204.47" y2="149.86" width="0.1524" layer="91"/>
-<label x="204.47" y="149.86" size="2.54" layer="95" rot="R270" xref="yes"/>
+<wire x1="196.85" y1="152.4" x2="196.85" y2="149.86" width="0.1524" layer="91"/>
+<label x="196.85" y="149.86" size="2.54" layer="95" rot="R270" xref="yes"/>
 </segment>
 <segment>
@@
 <segment>
 <pinref part="R9" gate="G$1" pin="1"/>
-<wire x1="194.31" y1="152.4" x2="194.31" y2="149.86" width="0.1524" layer="91"/>
-<label x="194.31" y="149.86" size="2.54" layer="95" rot="R270" xref="yes"/>
-</segment>
-<segment>
+<wire x1="186.69" y1="152.4" x2="186.69" y2="149.86" width="0.1524" layer="91"/>
+<label x="186.69" y="149.86" size="2.54" layer="95" rot="R270" xref="yes"/>
+</segment>
+<segment>
